Commit message: Added model for a green ball Changed the camera position from the bot to a new model i.e. a fixed stand Added the object detection and publisher node.

File: simulation/models/vehicle/macros.xacro (robot description, xacro)
@@ -5,5 +5,5 @@
         ixx="${m*(y*y+z*z)/12}" ixy = "0" ixz = "0"
         iyy="${m*(x*x+z*z)/12}" iyz = "0"
-        izz="${m*(x*x+z*z)/12}"
+        izz="${m*(x*x+y*y)/12}"
       />
   </xacro:macro>

File: simulation/models/vehicle/parameter.xacro (robot description, xacro)
@@ -13,5 +13,7 @@
   <xacro:property name="torque_wheel" value="10" />
   <xacro:property name="L_wheel" value="0.1788" />
+<!--
   <xacro:property name="cameraSize" value="0.05"/>
   <xacro:property name="cameraMass" value="0.1"/>
+-->
 </robot>

File: simulation/models/vehicle/vehicle.xacro (robot description, xacro)
@@ -124,5 +124,5 @@
   <!-- Set joints for the wheels which can be controlled over ROS -->
   <joint type="continuous" name="left_wheel_hinge">
-    <origin xyz="${-x_chassis/4} ${y_chassis/2+h_wheel/2} ${r_wheel/2-z_chassis/2}" rpy="0 0 0"/>
+    <origin xyz="${-x_chassis/3} ${y_chassis/2+h_wheel/2} ${r_wheel/2-z_chassis/2}" rpy="0 0 0"/>
     <child link="left_wheel"/>
     <parent link="base_link"/>
@@ -132,5 +132,5 @@
   </joint>
   <joint type="continuous" name="right_wheel_hinge">
-    <origin xyz="${-x_chassis/4} ${-y_chassis/2-h_wheel/2} ${r_wheel/2-z_chassis/2}" rpy="0 0 0"/>
+    <origin xyz="${-x_chassis/3} ${-y_chassis/2-h_wheel/2} ${r_wheel/2-z_chassis/2}" rpy="0 0 0"/>
     <child link="right_wheel"/>
     <parent link="base_link"/>
@@ -139,4 +139,5 @@
     <joint_properties damping="0.0" friction="0.0"/>
   </joint>
+<!--
   <link name="camera">
     <collision>
@@ -166,3 +167,4 @@
     <child link="camera"/>
   </joint>
+-->
 </robot>
