Commit message: Added walls on bot and changed camera orientation and position

File: simulation/models/fixed_camera/camera_parameter.xacro (robot description, xacro)
@@ -4,8 +4,8 @@
   <xacro:property name="cameraMass" value="0.1"/>
   <xacro:property name="x_camera" value="0" />
-  <xacro:property name="y_camera" value="-2" />
+  <xacro:property name="y_camera" value="-3" />
   <xacro:property name="z_camera" value="1" />
   <xacro:property name="x_stand" value="0" />
-  <xacro:property name="y_stand" value="-2.05" />
+  <xacro:property name="y_stand" value="-3.05" />
   <xacro:property name="z_stand" value="0.5225" />
   <xacro:property name="stand_xSize" value="0.1" />

File: simulation/models/fixed_camera/fixed_camera.xacro (robot description, xacro)
@@ -52,5 +52,5 @@
   </joint>
   <joint type="continuous" name="camera_stand_joint">
-    <origin xyz="${x_camera} ${y_camera} ${z_camera-cameraSize/2}" rpy="3.1429 3.1429 -1.5714"/>
+    <origin xyz="${x_camera} ${y_camera} ${z_camera-cameraSize/2}" rpy="0 -0.3 1.5714"/>
     <child link="camera"/>
     <parent link="stand"/>

File: simulation/models/vehicle/parameter.xacro (robot description, xacro)
@@ -17,3 +17,8 @@
   <xacro:property name="cameraMass" value="0.1"/>
 -->
+  <xacro:property name="wall_thickness" value="0.02" />
+  <xacro:property name="wall_height" value="0.1" />
+  <xacro:property name="wall_offset" value="0.025" />
+  <xacro:property name="wall_mass1" value="0.6" />
+  <xacro:property name="wall_mass2" value="0.9" />
 </robot>

File: simulation/models/vehicle/vehicle.xacro (robot description, xacro)
@@ -1,11 +1,8 @@
 <?xml version='1.0'?>
-<!-- choose a name space and start xacro -->
 <robot name="vehicle" xmlns:xacro="http://www.ros.org/wiki/xacro">
-  <!-- Start by including all required xacro files which hold the macros -->
   <xacro:include filename="$(find simulation)/models/vehicle/vehicle.gazebo" />
   <xacro:include filename="$(find simulation)/models/vehicle/materials.xacro"   />
   <xacro:include filename="$(find simulation)/models/vehicle/macros.xacro"      />
   <xacro:include filename="$(find simulation)/models/vehicle/parameter.xacro"   />
- <!-- Create a dummy link as base link -->
   <link name='base_link'>
     <pose>0 0 0 0 0 0</pose>
@@ -15,13 +12,10 @@
     <parent link="base_link"/>
   </joint>
-  <!-- Define the chassis of the differential drive robot, which is our base -->
   <link name='chassis_link'>
     <pose>0 0 0 0 0 0</pose>
-    <!-- Define inertial system for the chassis -->
     <inertial>
       <mass value="${m_chassis}"/>
       <xacro:box_inertia m="${m_chassis}" x="${x_chassis}" y="${y_chassis}" z="${z_chassis}"/>
     </inertial>
-    <!-- Define collision sorrounding box -->
     <collision name='collision'>
       <origin xyz="0 0 0" rpy=" 0 0 0"/>
@@ -30,5 +24,4 @@
       </geometry>
     </collision>
-    <!-- Define visualization structure -->
     <visual name='base_link_visual'>
 	  <origin xyz="0 0 0" rpy=" 0 0 0"/>
@@ -37,29 +30,53 @@
       </geometry>
     </visual>
-    <!-- Add the caster wheel! Here we simply assume complete slippage, thus we do not require that it rotates! -->
-    <collision name='caster_collision'>
-      <origin xyz="${-(r_wheel/2)+x_chassis/2} 0 ${-z_chassis/2}" rpy=" 0 0 0"/>
-      <geometry>
-        <sphere radius="${r_wheel/2}"/>
-      </geometry>
-      <surface>
-        <friction>
-          <ode>
-            <mu>0</mu>
-            <mu2>0</mu2>
-            <slip1>1.0</slip1>
-            <slip2>1.0</slip2>
-          </ode>
-        </friction>
-      </surface>
-    </collision>
-    <visual name='caster_visual'>
-      <origin xyz="${-(r_wheel/2)+x_chassis/2} 0 ${-z_chassis/2}" rpy=" 0 0 0"/>
-      <geometry>
-        <sphere radius="${r_wheel/2}"/>
-      </geometry>
-    </visual>
-  </link>
-  <!-- Add the wheels for the robot -->
+    <collision name='wall11_collision'>
+      <origin xyz="${-(x_chassis/2)+(wall_thickness/2)} 0 ${(z_chassis/2)+(wall_height/2)} " rpy=" 0 0 0"/>
+      <geometry>
+        <box size="${wall_thickness} ${y_chassis} ${wall_height}"/>
+      </geometry>
+    </collision>
+    <visual name='wall11_visual'>
+	  <origin xyz="${-(x_chassis/2)+(wall_thickness/2)} 0 ${(z_chassis/2)+(wall_height/2)}" rpy=" 0 0 0"/>
+      <geometry>
+        <box size="${wall_thickness} ${y_chassis} ${wall_height}"/>
+      </geometry>
+    </visual>
+    <collision name='wall12_collision'>
+      <origin xyz="${(x_chassis/2)-(wall_thickness/2)} 0 ${(z_chassis/2)+(wall_height/2)}" rpy=" 0 0 0"/>
+      <geometry>
+        <box size="${wall_thickness} ${y_chassis} ${wall_height}"/>
+      </geometry>
+    </collision>
+    <visual name='wall12_visual'>
+	    <origin xyz="${(x_chassis/2)-(wall_thickness/2)} 0 ${(z_chassis/2)+(wall_height/2)}" rpy=" 0 0 0"/>
+      <geometry>
+        <box size="${wall_thickness} ${y_chassis} ${wall_height}"/>
+      </geometry>
+    </visual>
+    <collision name='wall21_collision'>
+      <origin xyz="0 ${(y_chassis/2)-(wall_thickness/2)-wall_offset} ${(z_chassis/2)+(wall_height/2)}" rpy=" 0 0 0"/>
+      <geometry>
+        <box size="${x_chassis-2*wall_thickness} ${wall_thickness} ${wall_height}"/>
+      </geometry>
+    </collision>
+    <visual name='wall21_visual'>
+	  <origin xyz="0 ${(y_chassis/2)-(wall_thickness/2)-wall_offset} ${(z_chassis/2)+(wall_height/2)}" rpy=" 0 0 0"/>
+      <geometry>
+        <box size="${x_chassis-2*wall_thickness} ${wall_thickness} ${wall_height}"/>
+      </geometry>
+    </visual>
+    <collision name='wall22_collision'>
+      <origin xyz="0 ${-(y_chassis/2)+(wall_thickness/2)-wall_offset} ${(z_chassis/2)+(wall_height/2)}" rpy=" 0 0 0"/>
+      <geometry>
+        <box size="${x_chassis-2*wall_thickness} ${wall_thickness} ${wall_height}"/>
+      </geometry>
+    </collision>
+    <visual name='wall22_visual'>
+	  <origin xyz="0 ${-(y_chassis/2)+(wall_thickness/2)-wall_offset} ${(z_chassis/2)+(wall_height/2)}" rpy=" 0 0 0"/>
+      <geometry>
+        <box size="${x_chassis-2*wall_thickness} ${wall_thickness} ${wall_height}"/>
+      </geometry>
+    </visual>
+  </link>
   <link name="left_wheel">
     <collision name="collision">
@@ -122,5 +139,64 @@
     </inertial>
   </link>
-  <!-- Set joints for the wheels which can be controlled over ROS -->
+  <link name="right_wheel1">
+    <collision name="collision">
+      <origin xyz="0 0 0" rpy="0 1.5707 1.5707"/>
+      <geometry>
+        <cylinder radius="${r_wheel}" length="${h_wheel}"/>
+      </geometry>
+      <surface>
+        <friction>
+          <ode>
+            <mu>1.0</mu>
+            <mu2>1.0</mu2>
+            <slip1>0.0</slip1>
+            <slip2>0.0</slip2>
+          </ode>
+        </friction>
+      </surface>
+    </collision>
+    <visual name="right_wheel_visual">
+      <origin xyz="0 0 0" rpy="0 1.5707 1.5707"/>
+      <geometry>
+        <cylinder radius="${r_wheel}" length="${h_wheel}"/>
+      </geometry>
+    </visual>
+    <inertial>
+      <origin xyz="0 0 0" rpy="0 1.5707 1.5707"/>
+      <mass value="${m_wheel}"/>
+      <cylinder_inertia m="${m_wheel}" r="${r_wheel}" h="${h_wheel}"/>
+      <xacro:cylinder_inertia m="${m_wheel}" r="${r_wheel}" h="${h_wheel}"/>
+    </inertial>
+  </link>
+  <link name="left_wheel1">
+    <collision name="collision">
+      <origin xyz="0 0 0" rpy="0 1.5707 1.5707"/>
+      <geometry>
+        <cylinder radius="${r_wheel}" length="${h_wheel}"/>
+      </geometry>
+      <surface>
+        <friction>
+          <ode>
+            <mu>1.0</mu>
+            <mu2>1.0</mu2>
+            <slip1>0.0</slip1>
+            <slip2>0.0</slip2>
+          </ode>
+        </friction>
+      </surface>
+    </collision>
+    <visual name="left_wheel_visual">
+      <origin xyz="0 0 0" rpy="0 1.5707 1.5707"/>
+      <geometry>
+        <cylinder radius="${r_wheel}" length="${h_wheel}"/>
+      </geometry>
+    </visual>
+    <inertial>
+      <origin xyz="0 0 0" rpy="0 1.5707 1.5707"/>
+      <mass value="${m_wheel}"/>
+      <cylinder_inertia m="${m_wheel}" r="${r_wheel}" h="${h_wheel}"/>
+      <xacro:cylinder_inertia m="${m_wheel}" r="${r_wheel}" h="${h_wheel}"/>
+    </inertial>
+  </link>
   <joint type="continuous" name="left_wheel_hinge">
     <origin xyz="${-x_chassis/3} ${y_chassis/2+h_wheel/2} ${r_wheel/2-z_chassis/2}" rpy="0 0 0"/>
@@ -131,4 +207,12 @@
     <joint_properties damping="0.0" friction="0.0"/>
   </joint>
+  <joint type="continuous" name="left_wheel_hinge1">
+    <origin xyz="${+x_chassis/3} ${y_chassis/2+h_wheel/2} ${r_wheel/2-z_chassis/2}" rpy="0 0 0"/>
+    <child link="left_wheel1"/>
+    <parent link="base_link"/>
+    <axis xyz="0 1 0" rpy="0 0 0"/>
+    <limit effort="100" velocity="100"/>
+    <joint_properties damping="0.0" friction="0.0"/>
+  </joint>
   <joint type="continuous" name="right_wheel_hinge">
     <origin xyz="${-x_chassis/3} ${-y_chassis/2-h_wheel/2} ${r_wheel/2-z_chassis/2}" rpy="0 0 0"/>
@@ -139,32 +223,11 @@
     <joint_properties damping="0.0" friction="0.0"/>
   </joint>
-<!--
-  <link name="camera">
-    <collision>
-      <origin xyz="0 0 0" rpy="0 0 0"/>
-      <geometry>
-        <box size="${cameraSize} ${cameraSize} ${cameraSize}"/>
-      </geometry>
-    </collision>
-    <visual>
-      <origin xyz="0 0 0" rpy="0 0 0"/>
-      <geometry>
-        <box size="${cameraSize} ${cameraSize} ${cameraSize}"/>
-      </geometry>
-      <material name="green"/>
-    </visual>
-    <inertial>
-      <mass value="${cameraMass}" />
-      <origin xyz="0 0 0" rpy="0 0 0"/>
-      <box_inertia m="${cameraMass}" x="${cameraSize}" y="${cameraSize}" z="${cameraSize}" />
-      <inertia ixx="1e-6" ixy="0" ixz="0" iyy="1e-6" iyz="0" izz="1e-6" />
-    </inertial>
-  </link>
-  <joint name="camera_joint" type="fixed">
-    <axis xyz="0 1 0" />
-    <origin xyz="${x_chassis/2} 0 0" rpy="0 0 0"/>
-    <parent link="chassis_link"/>
-    <child link="camera"/>
-  </joint>
--->
+  <joint type="continuous" name="right_wheel_hinge1">
+    <origin xyz="${+x_chassis/3} ${-y_chassis/2-h_wheel/2} ${r_wheel/2-z_chassis/2}" rpy="0 0 0"/>
+    <child link="right_wheel1"/>
+    <parent link="base_link"/>
+    <axis xyz="0 1 0" rpy="0 0 0"/>
+    <limit effort="100" velocity="100"/>
+    <joint_properties damping="0.0" friction="0.0"/>
+  </joint>
 </robot>
