Commit message: Added "initial_velocity" plugin that gives initial velocity to an object. Changed "object" gazebo file to use the plugin Changed launch file to spawn the object

File: simulation/models/object/my_object.xacro (robot description, xacro)
@@ -25,5 +25,5 @@
 	  <origin xyz="0 0 2" rpy=" 0 0 0"/>
       <geometry>
-        <sphere radius="0.15"/>
+        <sphere radius="0.07"/>
       </geometry>
     </visual>
