Commit message: Added another camera(with stand) Added a node that subscribes both the cameras and publishes a dataset of 8 variables (4 from each camera) Added a node that subscribes the data set

File: simulation/models/fixed_camera_y/fixed_camera_y.xacro (robot description, xacro)
@@ -1,7 +1,7 @@
 <?xml version='1.0'?>
 <!-- choose a name space and start xacro -->
-<robot name="fixed_camera" xmlns:xacro="http://www.ros.org/wiki/xacro">
-  <xacro:include filename="$(find simulation)/models/fixed_camera/camera_parameter.xacro"   />
-  <xacro:include filename="$(find simulation)/models/fixed_camera/fixed_camera.gazebo" />
+<robot name="fixed_camera_y" xmlns:xacro="http://www.ros.org/wiki/xacro">
+  <xacro:include filename="$(find simulation)/models/fixed_camera_y/camera_parameter_y.xacro"   />
+  <xacro:include filename="$(find simulation)/models/fixed_camera_y/fixed_camera_y.gazebo" />
   <link name='base_link2'>
     <pose>${x_camera} ${y_camera} 0 0 0 0</pose>
@@ -52,5 +52,5 @@
   </joint>
   <joint type="continuous" name="camera_stand_joint">
-    <origin xyz="${x_camera} ${y_camera} ${z_camera-cameraSize/2}" rpy="0 -0.3 1.5714"/>
+    <origin xyz="${x_camera} ${y_camera} ${z_camera-cameraSize/2}" rpy="0 -0.3 0"/>
     <child link="camera"/>
     <parent link="stand"/>
